Commit message: Xacro transform fix (!), robot state publish frequency
* mount_body to hand_root static transform is shifted ~1 cm
* robot state is published too seldom if no specified frequency

File: models/ur5_allegro.xacro (robot description, xacro)
@@ -30,5 +30,5 @@
     <parent link="mount_body" />
     <child link = "hand_root" />
-    <origin xyz="0.0 0.0 0.0375" rpy="0.0 0.0 -0.79" />
+    <origin xyz="0.006 -0.006 0.0375" rpy="0.0 0.0 -0.79" />
   </joint>
 </robot>
