Commit message: Fixed Thumb URDF partially
J0 to J2 must be 55.4 mm in the hand manual p.19, but it was 57.6 mm in
the provided URDF file. J1-2 is 16.6.
I updated J0-1 and J1-2 values to sum upto 55.4 mm.
It is still not perfect: when the real thumb touches the palm,
visualized thumb does not touch it!

File: models/allegro_optoforce_right.xacro (robot description, xacro)
@@ -26,5 +26,5 @@
     <xacro:property name="link0_t_y" value="0.0340"/>
     <xacro:property name="link0_t_z" value="0.0455"/>
-    <xacro:property name="link1_t_z" value="0.0177"/>
+    <xacro:property name="link1_t_z" value="0.0166"/>
     <xacro:property name="link2_t_z" value="0.0514"/>
     <xacro:property name="link3_t_z" value="0.0313"/>
@@ -154,5 +154,5 @@
             <parent link="link_${finger_num*4+0}"/>
             <child link="link_${finger_num*4+1}"/>
-            <origin xyz="-0.027 0.005 0.0399"/>
+            <origin xyz="-0.027 0.005 0.0388"/>
             <dynamics damping="3" friction="5"/>
         </joint>

Commit message: Adapted to new ur5 driver package ur_robot_driver
* ur_modern_driver became obsolete
* changed default Moveit planner to BiTRRT
* created puppet.launch to play rosbags with simulation time.
* xacro file adjustments

File: models/allegro_optoforce_right.xacro (robot description, xacro)
@@ -26,5 +26,5 @@
     <xacro:property name="link0_t_y" value="0.0340"/>
     <xacro:property name="link0_t_z" value="0.0455"/>
-    <xacro:property name="link1_t_z" value="0.0166"/>
+    <xacro:property name="link1_t_z" value="0.0177"/>
     <xacro:property name="link2_t_z" value="0.0514"/>
     <xacro:property name="link3_t_z" value="0.0313"/>
@@ -154,5 +154,5 @@
             <parent link="link_${finger_num*4+0}"/>
             <child link="link_${finger_num*4+1}"/>
-            <origin xyz="-0.027 0.005 0.0388"/>
+            <origin xyz="-0.027 0.005 0.0399"/>
             <dynamics damping="3" friction="5"/>
         </joint>
@@ -230,5 +230,5 @@
             <parent link="link_${finger_num*4+3}"/>
             <child link="allegro_omd_adapter_${finger_num}"/>
-            <origin rpy="0 0 3.14" xyz="0 0 ${link3_t_z+adapter_offset}"/>
+            <origin rpy="0 0 3.14" xyz="0.001 0 ${link3_t_z+adapter_offset}"/>
         </joint>
     </xacro:macro>

File: models/ur5_allegro.xacro (robot description, xacro)
@@ -17,4 +17,5 @@
   <xacro:ur5_robot prefix="" joint_limited="false"
     transmission_hw_interface="$(arg transmission_hw_interface)"
+    kinematics_file="${load_yaml('$(arg kinematics_config)')}"
     />
   <!-- mount part connecting allegro to ur5-->
